File: Schematics/Bus-IO-and_Centronics-Card/Bus IO and Centronics Card.sch (EAGLE design)
At the start: 22 parts, among them IC1 W65C22S, IC2 74LS245N, IC3 7416N, X1 RJ45-8X

Commit message: Updated to have a formal Timer IRQ.  Currently this is T1 on the W65C22 on the GPIO card, so if you want to use it that card must be present.
The prebuilt ROM ToEVID.bin uses this card at 0xC040.

A couple of minor whoopsies have been fixed as well.
Parts:
- added D1, D3: BAT85, diode:BAT81
- renumbered SV1 to CENTRONICS_PORT, V1 to IC4, X1 to TPB
Connections:
- net PB3_TPB_RESET renamed PB3_TPB_SELECT
- new net PB0_ATN_OUT: IC1.PB0, IC3D.I
- net GND: now also D1.A, D3.A
- net PB2_TPB_ATN: now also IC3D.O
- net PB6_TPB_CLK: now also D3.C
- net PB7_TPB_DATA: now also D1.C
- net VCC: no longer IC3D.I
Other:
- moved on the sheet: C4, IC3B, IC3C, IC3D, IC3P
